Commit message: Add files via upload

File: jetbot/jetbot_description/urdf/jetbot.urdf (robot description, URDF)
Before this commit: robot jetbot, 4 links, 3 joints
Links:
- link chassis: mass 5 -> 10
- link left_wheel: mass 0.2 -> 0.3
- link right_wheel: mass 0.2 -> 0.3
Joints:
- joint left_wheel_hinge: limit lower=-1.6 upper=1.6 effort=10000000 velocity=0.7 -> lower=-1.6 upper=1.6 effort=100 velocity=100
- joint right_wheel_hinge: limit lower=-1.6 upper=1.6 effort=10000000 velocity=0.7 -> lower=-1.6 upper=1.6 effort=100 velocity=100
