Commit message: Add files via upload

File: jetbot/jetbot_description/urdf/jetbot.xacro (robot description, xacro)
@@ -1,5 +1,5 @@
 <?xml version="1.0"?>
 <robot name="jetbot" xmlns:xacro="http://www.ros.org/wiki/xacro">
-	<xacro:include filename="$(find my_robot_urdf)/urdf/jetbot.gazebo" />
+    <xacro:include filename="$(find my_robot_urdf)/urdf/jetbot.gazebo" />
     <link name="world"/>
     <joint name="fixed" type="fixed">
@@ -15,5 +15,5 @@
         <collision>
             <geometry>
-                <mesh filename="file://$(find my_robot_urdf)/urdf/jetbot/meshes/JetBot-v3-Chassis.dae" scale="0.001 0.001 0.001"/>
+                <mesh filename="file://$(find jetbot_description)/urdf/jetbot/meshes/JetBot-v3-Chassis.dae" scale="0.001 0.001 0.001"/>
             </geometry>
         </collision>
@@ -21,5 +21,5 @@
             <origin rpy="1.57079632679 0.0 1.57079632679" xyz="0.0 0.0 0.043"/>
             <geometry>
-                <mesh filename="file://$(find my_robot_urdf)/urdf/jetbot/meshes/JetBot-v3-Chassis.dae" scale="0.001 0.001 0.001"/>
+                <mesh filename="file://$(find jetbot_description)/urdf/jetbot/meshes/JetBot-v3-Chassis.dae" scale="0.001 0.001 0.001"/>
             </geometry>
         </visual>
@@ -34,5 +34,5 @@
             <origin rpy="0 0 0" xyz="0 0 0"/>
             <geometry>
-                <mesh filename="file://$(find my_robot_urdf)/urdf/jetbot/meshes/JetBot-v3-Wheel.stl" scale="0.001 0.001 0.001"/>
+                <mesh filename="file://$(find jetbot_description)/urdf/jetbot/meshes/JetBot-v3-Wheel.stl" scale="0.001 0.001 0.001"/>
             </geometry>
         </collision>
@@ -40,5 +40,5 @@
             <origin rpy="0 0 0" xyz="0 0 0"/>
             <geometry>
-                <mesh filename="file://$(find my_robot_urdf)/urdf/jetbot/meshes/JetBot-v3-Wheel.stl" scale="0.001 0.001 0.001"/>
+                <mesh filename="file://$(find jetbot_description)/urdf/jetbot/meshes/JetBot-v3-Wheel.stl" scale="0.001 0.001 0.001"/>
             </geometry>
         </visual>
@@ -49,5 +49,5 @@
         <parent link="chassis"/>
         <axis rpy="0 0 0" xyz="1 0 0"/>
-        <limit lower="-2.2" upper="0.7" effort="100" velocity="100"/>
+        <limit lower="0" upper="6.28319" effort="100" velocity="100"/>
     </joint>
     <link name="right_wheel">
@@ -60,5 +60,5 @@
             <origin rpy="0 0 0" xyz="0 0 0"/>
 	        <geometry>
-	            <mesh filename="file://$(find my_robot_urdf)/urdf/jetbot/meshes/JetBot-v3-Wheel.stl" scale="0.001 0.001 0.001"/>
+	            <mesh filename="file://$(find jetbot_description)/urdf/jetbot/meshes/JetBot-v3-Wheel.stl" scale="0.001 0.001 0.001"/>
 	        </geometry>
         </collision>
@@ -66,5 +66,5 @@
             <origin rpy="0 0 0" xyz="0 0 0"/>
 	        <geometry>
-	            <mesh filename="file://$(find my_robot_urdf)/urdf/jetbot/meshes/JetBot-v3-Wheel.stl" scale="0.001 0.001 0.001"/>
+	            <mesh filename="file://$(find jetbot_description)/urdf/jetbot/meshes/JetBot-v3-Wheel.stl" scale="0.001 0.001 0.001"/>
 	        </geometry>
 	    </visual>
@@ -75,5 +75,5 @@
         <parent link="chassis"/>
         <axis rpy="0 0 0" xyz="1 0 0"/>
-        <limit lower="-2.2" upper="0.7" effort="100" velocity="100"/>
+        <limit lower="0" upper="6.28319" effort="100" velocity="100"/>
     </joint>
     <link name="camera_link">

Commit message: Add files via upload

File: jetbot/jetbot_description/urdf/jetbot.xacro (robot description, xacro)
@@ -9,4 +9,5 @@
     <link name="chassis">
         <inertial>
+            <origin rpy="1.57079632679 0.0 1.57079632679" xyz="0.0 0.0 0.043"/>
             <mass value="5"/>
             <origin rpy="1.57079632679 0.0 1.57079632679" xyz="0.0 0.0 0.043"/>
@@ -14,4 +15,5 @@
         </inertial>
         <collision>
+            <origin rpy="1.57079632679 0.0 1.57079632679" xyz="0.0 0.0 0.043"/>
             <geometry>
                 <mesh filename="file://$(find jetbot_description)/urdf/jetbot/meshes/JetBot-v3-Chassis.dae" scale="0.001 0.001 0.001"/>

Commit message: Add files via upload

File: jetbot/jetbot_description/urdf/jetbot.xacro (robot description, xacro)
@@ -2,15 +2,21 @@
 <robot name="jetbot" xmlns:xacro="http://www.ros.org/wiki/xacro">
     <xacro:include filename="$(find my_robot_urdf)/urdf/jetbot.gazebo" />
-    <link name="world"/>
-    <joint name="fixed" type="fixed">
-        <parent link="world"/>
-        <child link="chassis"/>
-    </joint>
+    <xacro:property name="follow_wheel_radius" value="0.0135"/>
+    <xacro:property name="follow_wheel_length" value="0.011"/>
+    <xacro:property name="follow_wheel_mass" value="0.66"/>
+    <xacro:macro name="cylinder_inertial" params="radius length mass *origin">
+      <inertial>
+        <mass value="${mass}" />
+        <xacro:insert_block name="origin" />
+        <inertia ixx="${0.0833333 * mass * (3 * radius * radius + length * length)}" ixy="0.0" ixz="0.0"
+          iyy="${0.0833333 * mass * (3 * radius * radius + length * length)}" iyz="0.0"
+          izz="${0.5 * mass * radius * radius}" />
+      </inertial>
+    </xacro:macro>
     <link name="chassis">
         <inertial>
             <origin rpy="1.57079632679 0.0 1.57079632679" xyz="0.0 0.0 0.043"/>
-            <mass value="5"/>
-            <origin rpy="1.57079632679 0.0 1.57079632679" xyz="0.0 0.0 0.043"/>
-            <inertia ixx="0.0395416666667" ixy="0" ixz="0" iyy="0.106208333333" iyz="0" izz="0.106208333333"/>
+            <mass value="50"/>
+            <inertia ixx="10"  ixy="0"  ixz="0" iyy="8" iyz="0" izz="6" />
         </inertial>
         <collision>
@@ -29,7 +35,7 @@
     <link name="left_wheel">
         <inertial>
-            <mass value="0.2"/>
+            <mass value="10"/>
             <origin rpy="0 0 0" xyz="0 0 0"/>
-            <inertia ixx="0" ixy="0" ixz="0" iyy="0" iyz="0" izz="0"/>
+            <inertia ixx="1"  ixy="0"  ixz="0" iyy="8" iyz="0" izz="6" />
         </inertial>
         <collision>
@@ -38,4 +44,13 @@
                 <mesh filename="file://$(find jetbot_description)/urdf/jetbot/meshes/JetBot-v3-Wheel.stl" scale="0.001 0.001 0.001"/>
             </geometry>
+            <surface>
+                <friction>
+                    <torsional>
+                        <coefficient>10000.0</coefficient>
+                        <surface_radius>0.5</surface_radius>
+                        <use_patch_radius>false</use_patch_radius>
+                    </torsional>
+                </friction>
+            </surface>
         </collision>
 	    <visual>
@@ -51,11 +66,11 @@
         <parent link="chassis"/>
         <axis rpy="0 0 0" xyz="1 0 0"/>
-        <limit lower="0" upper="6.28319" effort="100" velocity="100"/>
+        <limit lower="-360" upper="360" effort="10" velocity="10"/>
     </joint>
     <link name="right_wheel">
         <inertial>
-            <mass value="0.2"/>
+            <mass value="10"/>
             <origin rpy="0 0 0" xyz="0 0 0"/>
-            <inertia ixx="0" ixy="0" ixz="0" iyy="0" iyz="0" izz="0"/>
+            <inertia ixx="1" ixy="0" ixz="0" iyy="8" iyz="0" izz="6" />
         </inertial>
         <collision>
@@ -64,11 +79,20 @@
 	            <mesh filename="file://$(find jetbot_description)/urdf/jetbot/meshes/JetBot-v3-Wheel.stl" scale="0.001 0.001 0.001"/>
 	        </geometry>
+            <surface>
+                <friction>
+                    <torsional>
+                        <coefficient>10000.0</coefficient>
+                        <surface_radius>0.5</surface_radius>
+                        <use_patch_radius>false</use_patch_radius>
+                    </torsional>
+                </friction>
+            </surface>
         </collision>
-	    <visual>
-            <origin rpy="0 0 0" xyz="0 0 0"/>
-	        <geometry>
-	            <mesh filename="file://$(find jetbot_description)/urdf/jetbot/meshes/JetBot-v3-Wheel.stl" scale="0.001 0.001 0.001"/>
-	        </geometry>
-	    </visual>
+	<visual>
+        <origin rpy="0 0 0" xyz="0 0 0"/>
+	    <geometry>
+	        <mesh filename="file://$(find jetbot_description)/urdf/jetbot/meshes/JetBot-v3-Wheel.stl" scale="0.001 0.001 0.001"/>
+	    </geometry>
+	</visual>
     </link>
     <joint name='right_wheel_hinge' type='revolute'>
@@ -77,5 +101,5 @@
         <parent link="chassis"/>
         <axis rpy="0 0 0" xyz="1 0 0"/>
-        <limit lower="0" upper="6.28319" effort="100" velocity="100"/>
+        <limit lower="-360" upper="360" effort="10" velocity="10"/>
     </joint>
     <link name="camera_link">

Commit message: Add files via upload

File: jetbot/jetbot_description/urdf/jetbot.xacro (robot description, xacro)
@@ -16,18 +16,18 @@
     <link name="chassis">
         <inertial>
-            <origin rpy="1.57079632679 0.0 1.57079632679" xyz="0.0 0.0 0.043"/>
+            <origin rpy="1.57079632679 0.0 1.57079632679" xyz="0.0 0.0 0.084"/>
             <mass value="50"/>
-            <inertia ixx="10"  ixy="0"  ixz="0" iyy="8" iyz="0" izz="6" />
+            <inertia ixx="1"  ixy="0"  ixz="0" iyy="0.8" iyz="0" izz="0.6" />
         </inertial>
         <collision>
-            <origin rpy="1.57079632679 0.0 1.57079632679" xyz="0.0 0.0 0.043"/>
+            <origin rpy="1.57079632679 0.0 1.57079632679" xyz="0.0 0.0 0.084"/>
             <geometry>
-                <mesh filename="file://$(find jetbot_description)/urdf/jetbot/meshes/JetBot-v3-Chassis.dae" scale="0.001 0.001 0.001"/>
+                <mesh filename="file://$(find jetbot_description)/urdf/jetbot/meshes/JetBot-v3-Chassis.dae" scale="0.002 0.002 0.002"/>
             </geometry>
         </collision>
         <visual>
-            <origin rpy="1.57079632679 0.0 1.57079632679" xyz="0.0 0.0 0.043"/>
+            <origin rpy="1.57079632679 0.0 1.57079632679" xyz="0.0 0.0 0.084"/>
             <geometry>
-                <mesh filename="file://$(find jetbot_description)/urdf/jetbot/meshes/JetBot-v3-Chassis.dae" scale="0.001 0.001 0.001"/>
+                <mesh filename="file://$(find jetbot_description)/urdf/jetbot/meshes/JetBot-v3-Chassis.dae" scale="0.002 0.002 0.002"/>
             </geometry>
         </visual>
@@ -35,5 +35,5 @@
     <link name="left_wheel">
         <inertial>
-            <mass value="10"/>
+            <mass value="5"/>
             <origin rpy="0 0 0" xyz="0 0 0"/>
             <inertia ixx="1"  ixy="0"  ixz="0" iyy="8" iyz="0" izz="6" />
@@ -42,5 +42,5 @@
             <origin rpy="0 0 0" xyz="0 0 0"/>
             <geometry>
-                <mesh filename="file://$(find jetbot_description)/urdf/jetbot/meshes/JetBot-v3-Wheel.stl" scale="0.001 0.001 0.001"/>
+                <mesh filename="file://$(find jetbot_description)/urdf/jetbot/meshes/JetBot-v3-Wheel.stl" scale="0.002 0.002 0.002"/>
             </geometry>
             <surface>
@@ -57,10 +57,10 @@
             <origin rpy="0 0 0" xyz="0 0 0"/>
             <geometry>
-                <mesh filename="file://$(find jetbot_description)/urdf/jetbot/meshes/JetBot-v3-Wheel.stl" scale="0.001 0.001 0.001"/>
+                <mesh filename="file://$(find jetbot_description)/urdf/jetbot/meshes/JetBot-v3-Wheel.stl" scale="0.002 0.002 0.002"/>
             </geometry>
         </visual>
     </link>
     <joint name='left_wheel_hinge' type='revolute'>
-        <origin rpy="0.0 0.0 1.57079632679" xyz="0.03 0.05125 0.03"/>
+        <origin rpy="0.0 0.0 1.57079632679" xyz="0.06 0.1025 0.06"/>
         <child  link="left_wheel"/>
         <parent link="chassis"/>
@@ -70,5 +70,5 @@
     <link name="right_wheel">
         <inertial>
-            <mass value="10"/>
+            <mass value="5"/>
             <origin rpy="0 0 0" xyz="0 0 0"/>
             <inertia ixx="1" ixy="0" ixz="0" iyy="8" iyz="0" izz="6" />
@@ -77,5 +77,5 @@
             <origin rpy="0 0 0" xyz="0 0 0"/>
 	        <geometry>
-	            <mesh filename="file://$(find jetbot_description)/urdf/jetbot/meshes/JetBot-v3-Wheel.stl" scale="0.001 0.001 0.001"/>
+	            <mesh filename="file://$(find jetbot_description)/urdf/jetbot/meshes/JetBot-v3-Wheel.stl" scale="0.002 0.002 0.002"/>
 	        </geometry>
             <surface>
@@ -90,12 +90,12 @@
         </collision>
 	<visual>
-        <origin rpy="0 0 0" xyz="0 0 0"/>
+            <origin rpy="0 0 0" xyz="0 0 0"/>
 	    <geometry>
-	        <mesh filename="file://$(find jetbot_description)/urdf/jetbot/meshes/JetBot-v3-Wheel.stl" scale="0.001 0.001 0.001"/>
+	        <mesh filename="file://$(find jetbot_description)/urdf/jetbot/meshes/JetBot-v3-Wheel.stl" scale="0.002 0.002 0.002"/>
 	    </geometry>
 	</visual>
     </link>
     <joint name='right_wheel_hinge' type='revolute'>
-        <origin rpy="0.0 0.0 1.57079632679 " xyz="0.03 -0.0595 0.03"/>
+        <origin rpy="0.0 0.0 1.57079632679 " xyz="0.06 -0.1025 0.06"/>
         <child  link="right_wheel"/>
         <parent link="chassis"/>
@@ -104,23 +104,24 @@
     </joint>
     <link name="camera_link">
+        <gravity>false</gravity>
         <inertial>
-            <origin xyz="0 0 0" rpy="0 0 0"/>
-            <mass value="0.1" />
-            <inertia ixx="1e-6" ixy="0" ixz="0" iyy="1e-6" iyz="0" izz="1e-6" />
+            <inertia ixx="1" ixy="0" ixz="0" iyy="8" iyz="0" izz="6" />
+	    <mass value="1"/>
         </inertial>
-        <visual>
+        <visual name="visual">
+            <origin rpy="0 0 0" xyz="0 0.0 0"/>
             <geometry>
-                <box size="0.001 0.001 0.001"/>
+                <box size="0.002 0.002 0.002"/>
             </geometry>
-            <material name="blue">
-                <color rgba="0 0 1.0 1.0"/>
-            </material>
         </visual>
     </link>
     <joint name="camera_joint" type="fixed">
+        <origin rpy="0 0.25 0" xyz="0.11 0.0 0.1714"/>
+        <child  link="camera_link"/>
         <parent link="chassis"/>
-        <child link="camera_link"/>
-        <origin rpy="0 0 0" xyz="0.047 0.0 0.0"/>
-        <axis xyz="1 0 0" />
+        <pose>0.0 0.0 0.0 0.0 0.0 0.0</pose>
+        <axis>
+            <xyz>0.1 0.0 0.0</xyz>
+        </axis>
     </joint>
     <transmission name="tran1">

Commit message: Add files via upload

File: jetbot/jetbot_description/urdf/jetbot.xacro (robot description, xacro)
@@ -1,5 +1,5 @@
 <?xml version="1.0"?>
 <robot name="jetbot" xmlns:xacro="http://www.ros.org/wiki/xacro">
-    <xacro:include filename="$(find my_robot_urdf)/urdf/jetbot.gazebo" />
+    <xacro:include filename="$(find jetbot_description)/urdf/jetbot.gazebo" />
     <xacro:property name="follow_wheel_radius" value="0.0135"/>
     <xacro:property name="follow_wheel_length" value="0.011"/>
@@ -15,114 +15,106 @@
     </xacro:macro>
     <link name="chassis">
-        <inertial>
-            <origin rpy="1.57079632679 0.0 1.57079632679" xyz="0.0 0.0 0.084"/>
-            <mass value="50"/>
-            <inertia ixx="1"  ixy="0"  ixz="0" iyy="0.8" iyz="0" izz="0.6" />
-        </inertial>
-        <collision>
-            <origin rpy="1.57079632679 0.0 1.57079632679" xyz="0.0 0.0 0.084"/>
-            <geometry>
-                <mesh filename="file://$(find jetbot_description)/urdf/jetbot/meshes/JetBot-v3-Chassis.dae" scale="0.002 0.002 0.002"/>
-            </geometry>
-        </collision>
-        <visual>
-            <origin rpy="1.57079632679 0.0 1.57079632679" xyz="0.0 0.0 0.084"/>
-            <geometry>
-                <mesh filename="file://$(find jetbot_description)/urdf/jetbot/meshes/JetBot-v3-Chassis.dae" scale="0.002 0.002 0.002"/>
-            </geometry>
-        </visual>
+      <inertial>
+        <origin rpy="1.57079632679 0.0 1.57079632679" xyz="0.0 0.0 0.086"/>
+        <mass value="50"/>
+        <inertia ixx="0"  ixy="0"  ixz="0" iyy="0" iyz="0" izz="0" />
+      </inertial>
+      <collision>
+        <origin rpy="1.57079632679 0.0 1.57079632679" xyz="0.0 0.0 0.086"/>
+        <geometry>
+          <mesh filename="file://$(find jetbot_description)/urdf/jetbot/meshes/JetBot-v3-Chassis.dae" scale="0.002 0.002 0.002"/>
+        </geometry>
+      </collision>
+      <visual>
+        <origin rpy="1.57079632679 0.0 1.57079632679" xyz="0.0 0.0 0.086"/>
+        <geometry>
+          <mesh filename="file://$(find jetbot_description)/urdf/jetbot/meshes/JetBot-v3-Chassis.dae" scale="0.002 0.002 0.002"/>
+        </geometry>
+      </visual>
     </link>
     <link name="left_wheel">
-        <inertial>
-            <mass value="5"/>
-            <origin rpy="0 0 0" xyz="0 0 0"/>
-            <inertia ixx="1"  ixy="0"  ixz="0" iyy="8" iyz="0" izz="6" />
-        </inertial>
-        <collision>
-            <origin rpy="0 0 0" xyz="0 0 0"/>
-            <geometry>
-                <mesh filename="file://$(find jetbot_description)/urdf/jetbot/meshes/JetBot-v3-Wheel.stl" scale="0.002 0.002 0.002"/>
-            </geometry>
-            <surface>
-                <friction>
-                    <torsional>
-                        <coefficient>10000.0</coefficient>
-                        <surface_radius>0.5</surface_radius>
-                        <use_patch_radius>false</use_patch_radius>
-                    </torsional>
-                </friction>
-            </surface>
-        </collision>
-	    <visual>
-            <origin rpy="0 0 0" xyz="0 0 0"/>
-            <geometry>
-                <mesh filename="file://$(find jetbot_description)/urdf/jetbot/meshes/JetBot-v3-Wheel.stl" scale="0.002 0.002 0.002"/>
-            </geometry>
-        </visual>
+      <inertial>
+        <mass value="1"/>
+        <origin rpy="0 0 0" xyz="0 0 0"/>
+        <inertia ixx="0"  ixy="0"  ixz="0" iyy="0" iyz="0" izz="0" />
+      </inertial>
+      <collision>
+        <origin rpy="0 0 0" xyz="0 0 0"/>
+        <geometry>
+          <mesh filename="file://$(find jetbot_description)/urdf/jetbot/meshes/JetBot-v3-Wheel.stl" scale="0.002 0.002 0.002"/>
+        </geometry>
+      </collision>
+      <visual>
+        <origin rpy="0 0 0" xyz="0 0 0"/>
+          <geometry>
+            <mesh filename="file://$(find jetbot_description)/urdf/jetbot/meshes/JetBot-v3-Wheel.stl" scale="0.002 0.002 0.002"/>
+          </geometry>
+      </visual>
     </link>
     <joint name='left_wheel_hinge' type='revolute'>
-        <origin rpy="0.0 0.0 1.57079632679" xyz="0.06 0.1025 0.06"/>
-        <child  link="left_wheel"/>
-        <parent link="chassis"/>
-        <axis rpy="0 0 0" xyz="1 0 0"/>
-        <limit lower="-360" upper="360" effort="10" velocity="10"/>
+      <origin rpy="0.0 0.0 1.57079632679" xyz="0.06 0.1025 0.06"/>
+      <child  link="left_wheel"/>
+      <parent link="chassis"/>
+      <axis rpy="0 0 0" xyz="1 0 0"/>
+      <limit lower="-360" upper="360" effort="50" velocity="100"/>
     </joint>
     <link name="right_wheel">
-        <inertial>
-            <mass value="5"/>
-            <origin rpy="0 0 0" xyz="0 0 0"/>
-            <inertia ixx="1" ixy="0" ixz="0" iyy="8" iyz="0" izz="6" />
-        </inertial>
-        <collision>
-            <origin rpy="0 0 0" xyz="0 0 0"/>
-	        <geometry>
-	            <mesh filename="file://$(find jetbot_description)/urdf/jetbot/meshes/JetBot-v3-Wheel.stl" scale="0.002 0.002 0.002"/>
-	        </geometry>
-            <surface>
-                <friction>
-                    <torsional>
-                        <coefficient>10000.0</coefficient>
-                        <surface_radius>0.5</surface_radius>
-                        <use_patch_radius>false</use_patch_radius>
-                    </torsional>
-                </friction>
-            </surface>
-        </collision>
-	<visual>
-            <origin rpy="0 0 0" xyz="0 0 0"/>
-	    <geometry>
-	        <mesh filename="file://$(find jetbot_description)/urdf/jetbot/meshes/JetBot-v3-Wheel.stl" scale="0.002 0.002 0.002"/>
-	    </geometry>
-	</visual>
+      <inertial>
+        <mass value="1"/>
+        <origin rpy="0 0 0" xyz="0 0 0"/>
+        <inertia ixx="0"  ixy="0"  ixz="0" iyy="0" iyz="0" izz="0" />
+      </inertial>
+      <collision>
+        <origin rpy="0 0 0" xyz="0 0 0"/>
+        <geometry>
+          <mesh filename="file://$(find jetbot_description)/urdf/jetbot/meshes/JetBot-v3-Wheel.stl" scale="0.002 0.002 0.002"/>
+        </geometry>
+      </collision>
+      <visual>
+        <origin rpy="0 0 0" xyz="0 0 0"/>
+        <geometry>
+          <mesh filename="file://$(find jetbot_description)/urdf/jetbot/meshes/JetBot-v3-Wheel.stl" scale="0.002 0.002 0.002"/>
+        </geometry>
+      </visual>
     </link>
     <joint name='right_wheel_hinge' type='revolute'>
-        <origin rpy="0.0 0.0 1.57079632679 " xyz="0.06 -0.1025 0.06"/>
-        <child  link="right_wheel"/>
-        <parent link="chassis"/>
-        <axis rpy="0 0 0" xyz="1 0 0"/>
-        <limit lower="-360" upper="360" effort="10" velocity="10"/>
+      <origin rpy="0.0 0.0 1.57079632679 " xyz="0.06 -0.119 0.06"/>
+      <child  link="right_wheel"/>
+      <parent link="chassis"/>
+      <axis rpy="0 0 0" xyz="1 0 0"/>
+      <limit lower="-360" upper="360" effort="50" velocity="100"/>
     </joint>
+    <joint name="camera_joint" type="fixed">
+      <origin rpy="0 0.25 0" xyz="0.11 0.0 0.1714"/>
+      <child  link="camera_link"/>
+      <parent link="chassis"/>
+      <pose>0.0 0.0 0.0 0.0 0.0 0.0</pose>
+      <axis>
+        <xyz>0.1 0.0 0.0</xyz>
+      </axis>
+    </joint>
+    <!-- Camera -->
     <link name="camera_link">
-        <gravity>false</gravity>
-        <inertial>
-            <inertia ixx="1" ixy="0" ixz="0" iyy="8" iyz="0" izz="6" />
-	    <mass value="1"/>
-        </inertial>
-        <visual name="visual">
-            <origin rpy="0 0 0" xyz="0 0.0 0"/>
-            <geometry>
-                <box size="0.002 0.002 0.002"/>
-            </geometry>
-        </visual>
+      <gravity>false</gravity>
+      <inertial>
+        <inertia ixx="0"  ixy="0"  ixz="0" iyy="0" iyz="0" izz="0" />
+        <mass value="1"/>
+      </inertial>
+      <visual name="visual">
+        <origin rpy="0 0 0" xyz="0 0.0 0"/>
+        <geometry>
+          <box size="0.002 0.002 0.002"/>
+        </geometry>
+      </visual>
     </link>
-    <joint name="camera_joint" type="fixed">
-        <origin rpy="0 0.25 0" xyz="0.11 0.0 0.1714"/>
-        <child  link="camera_link"/>
-        <parent link="chassis"/>
-        <pose>0.0 0.0 0.0 0.0 0.0 0.0</pose>
-        <axis>
-            <xyz>0.1 0.0 0.0</xyz>
-        </axis>
+    <joint name="camera_optical_joint" type="fixed">
+      <!-- these values have to be these values otherwise the gazebo camera image
+          won't be aligned properly with the frame it is supposedly originating from -->
+      <origin xyz="0 0 0" rpy="0 0 0"/>
+      <parent link="camera_link"/>
+      <child link="camera_link_optical"/>
     </joint>
+    <link name="camera_link_optical">
+    </link>
     <transmission name="tran1">
       <type>transmission_interface/SimpleTransmission</type>
