Commit message: Add files via upload

File: jetbot/jetbot_description/urdf/jetbot.xacro (robot description, xacro)
@@ -17,6 +17,6 @@
       <inertial>
         <origin rpy="1.57079632679 0.0 1.57079632679" xyz="0.0 0.0 0.086"/>
-        <mass value="50"/>
-        <inertia ixx="0"  ixy="0"  ixz="0" iyy="0" iyz="0" izz="0" />
+        <mass value="100"/>
+        <inertia ixx="0.001" ixy="0.001" ixz="0.001" iyy="0.001" iyz="0.001" izz="0.001" />
       </inertial>
       <collision>
@@ -35,7 +35,7 @@
     <link name="left_wheel">
       <inertial>
-        <mass value="1"/>
         <origin rpy="0 0 0" xyz="0 0 0"/>
-        <inertia ixx="0"  ixy="0"  ixz="0" iyy="0" iyz="0" izz="0" />
+        <mass value="5"/>
+        <inertia ixx="0.01" ixy="0.01" ixz="0.01" iyy="0.01" iyz="0.01" izz="0.01" />
       </inertial>
       <collision>
@@ -57,11 +57,12 @@
       <parent link="chassis"/>
       <axis rpy="0 0 0" xyz="1 0 0"/>
-      <limit lower="-360" upper="360" effort="50" velocity="100"/>
+      <limit lower="-1e+16" upper="1e+16" effort="200" velocity="100"/>
     </joint>
     <link name="right_wheel">
       <inertial>
+        <origin rpy="0 0 0" xyz="0 0 0"/>
+        <mass value="5"/>
+        <inertia ixx="0.01" ixy="0.01" ixz="0.01" iyy="0.01" iyz="0.01" izz="0.01" />
         <mass value="1"/>
-        <origin rpy="0 0 0" xyz="0 0 0"/>
-        <inertia ixx="0"  ixy="0"  ixz="0" iyy="0" iyz="0" izz="0" />
       </inertial>
       <collision>
@@ -83,5 +84,5 @@
       <parent link="chassis"/>
       <axis rpy="0 0 0" xyz="1 0 0"/>
-      <limit lower="-360" upper="360" effort="50" velocity="100"/>
+      <limit lower="-1e+16" upper="1e+16" effort="200" velocity="100"/>
     </joint>
     <joint name="camera_joint" type="fixed">
@@ -99,5 +100,5 @@
       <inertial>
         <inertia ixx="0"  ixy="0"  ixz="0" iyy="0" iyz="0" izz="0" />
-        <mass value="1"/>
+        <mass value="0.1"/>
       </inertial>
       <visual name="visual">

Commit message: Add files via upload
Find stable model parameter

File: jetbot/jetbot_description/urdf/jetbot.xacro (robot description, xacro)
@@ -17,5 +17,5 @@
       <inertial>
         <origin rpy="1.57079632679 0.0 1.57079632679" xyz="0.0 0.0 0.086"/>
-        <mass value="100"/>
+        <mass value="50"/>
         <inertia ixx="0.001" ixy="0.001" ixz="0.001" iyy="0.001" iyz="0.001" izz="0.001" />
       </inertial>
@@ -36,6 +36,6 @@
       <inertial>
         <origin rpy="0 0 0" xyz="0 0 0"/>
-        <mass value="5"/>
-        <inertia ixx="0.01" ixy="0.01" ixz="0.01" iyy="0.01" iyz="0.01" izz="0.01" />
+        <mass value="3"/>
+        <inertia ixx="0.001" ixy="0.001" ixz="0.001" iyy="0.001" iyz="0.001" izz="0.001" />
       </inertial>
       <collision>
@@ -62,6 +62,6 @@
       <inertial>
         <origin rpy="0 0 0" xyz="0 0 0"/>
-        <mass value="5"/>
-        <inertia ixx="0.01" ixy="0.01" ixz="0.01" iyy="0.01" iyz="0.01" izz="0.01" />
+        <mass value="3"/>
+        <inertia ixx="0.001" ixy="0.001" ixz="0.001" iyy="0.001" iyz="0.001" izz="0.001" />
         <mass value="1"/>
       </inertial>

Commit message: Add files via upload
Phisical Parameter Update

File: jetbot/jetbot_description/urdf/jetbot.xacro (robot description, xacro)
@@ -2,21 +2,9 @@
 <robot name="jetbot" xmlns:xacro="http://www.ros.org/wiki/xacro">
     <xacro:include filename="$(find jetbot_description)/urdf/jetbot.gazebo" />
-    <xacro:property name="follow_wheel_radius" value="0.0135"/>
-    <xacro:property name="follow_wheel_length" value="0.011"/>
-    <xacro:property name="follow_wheel_mass" value="0.66"/>
-    <xacro:macro name="cylinder_inertial" params="radius length mass *origin">
-      <inertial>
-        <mass value="${mass}" />
-        <xacro:insert_block name="origin" />
-        <inertia ixx="${0.0833333 * mass * (3 * radius * radius + length * length)}" ixy="0.0" ixz="0.0"
-          iyy="${0.0833333 * mass * (3 * radius * radius + length * length)}" iyz="0.0"
-          izz="${0.5 * mass * radius * radius}" />
-      </inertial>
-    </xacro:macro>
     <link name="chassis">
       <inertial>
-        <origin rpy="1.57079632679 0.0 1.57079632679" xyz="0.0 0.0 0.086"/>
-        <mass value="50"/>
-        <inertia ixx="0.001" ixy="0.001" ixz="0.001" iyy="0.001" iyz="0.001" izz="0.001" />
+        <mass value="10"/>
+        <origin rpy="0 0 0" xyz="0 0 0"/>
+        <inertia ixx="0.08025" ixy="0" ixz="0" iyy="0.08025" iyz="0" izz="0.1445"/>
       </inertial>
       <collision>
@@ -35,7 +23,7 @@
     <link name="left_wheel">
       <inertial>
-        <origin rpy="0 0 0" xyz="0 0 0"/>
-        <mass value="3"/>
-        <inertia ixx="0.001" ixy="0.001" ixz="0.001" iyy="0.001" iyz="0.001" izz="0.001" />
+        <mass value="0.3"/>
+        <origin rpy="0 1.5707 1.5707" xyz="0 0 0"/>
+        <inertia ixx="0.000129167" ixy="0" ixz="0" iyy="0.000129167" iyz="0" izz="0.0000225"/>
       </inertial>
       <collision>
@@ -57,12 +45,11 @@
       <parent link="chassis"/>
       <axis rpy="0 0 0" xyz="1 0 0"/>
-      <limit lower="-1e+16" upper="1e+16" effort="200" velocity="100"/>
+      <limit lower="-1e+16" upper="1e+16" effort="1000" velocity="100"/>
     </joint>
     <link name="right_wheel">
       <inertial>
-        <origin rpy="0 0 0" xyz="0 0 0"/>
-        <mass value="3"/>
-        <inertia ixx="0.001" ixy="0.001" ixz="0.001" iyy="0.001" iyz="0.001" izz="0.001" />
-        <mass value="1"/>
+        <mass value="0.3"/>
+        <origin rpy="0 1.5707 1.5707" xyz="0 0 0"/>
+        <inertia ixx="0.000129167" ixy="0" ixz="0" iyy="0.000129167" iyz="0" izz="0.0000225"/>
       </inertial>
       <collision>
@@ -84,5 +71,5 @@
       <parent link="chassis"/>
       <axis rpy="0 0 0" xyz="1 0 0"/>
-      <limit lower="-1e+16" upper="1e+16" effort="200" velocity="100"/>
+      <limit lower="-1e+16" upper="1e+16" effort="1000" velocity="100"/>
     </joint>
     <joint name="camera_joint" type="fixed">

Commit message: Add files via upload
Transmission is changed from effort to velocity

File: jetbot/jetbot_description/urdf/jetbot.xacro (robot description, xacro)
@@ -4,5 +4,5 @@
     <link name="chassis">
       <inertial>
-        <mass value="10"/>
+        <mass value="2.0"/>
         <origin rpy="0 0 0" xyz="0 0 0"/>
         <inertia ixx="0.08025" ixy="0" ixz="0" iyy="0.08025" iyz="0" izz="0.1445"/>
@@ -24,5 +24,5 @@
       <inertial>
         <mass value="0.3"/>
-        <origin rpy="0 1.5707 1.5707" xyz="0 0 0"/>
+        <origin rpy="0 0 0" xyz="0 0 0"/>
         <inertia ixx="0.000129167" ixy="0" ixz="0" iyy="0.000129167" iyz="0" izz="0.0000225"/>
       </inertial>
@@ -45,10 +45,10 @@
       <parent link="chassis"/>
       <axis rpy="0 0 0" xyz="1 0 0"/>
-      <limit lower="-1e+16" upper="1e+16" effort="1000" velocity="100"/>
+      <limit lower="-1e+16" upper="1e+16" effort="100" velocity="100"/>
     </joint>
     <link name="right_wheel">
       <inertial>
         <mass value="0.3"/>
-        <origin rpy="0 1.5707 1.5707" xyz="0 0 0"/>
+        <origin rpy="0 0 0" xyz="0 0 0"/>
         <inertia ixx="0.000129167" ixy="0" ixz="0" iyy="0.000129167" iyz="0" izz="0.0000225"/>
       </inertial>
@@ -71,5 +71,5 @@
       <parent link="chassis"/>
       <axis rpy="0 0 0" xyz="1 0 0"/>
-      <limit lower="-1e+16" upper="1e+16" effort="1000" velocity="100"/>
+      <limit lower="-1e+16" upper="1e+16" effort="100" velocity="100"/>
     </joint>
     <joint name="camera_joint" type="fixed">
@@ -108,8 +108,8 @@
       <type>transmission_interface/SimpleTransmission</type>
       <joint name="left_wheel_hinge">
-        <hardwareInterface>hardware_interface/EffortJointInterface</hardwareInterface>
+        <hardwareInterface>hardware_interface/VelocityJointInterface</hardwareInterface>
       </joint>
       <actuator name="motor1">
-        <hardwareInterface>hardware_interface/EffortJointInterface</hardwareInterface>
+        <hardwareInterface>hardware_interface/VelocityJointInterface</hardwareInterface>
         <mechanicalReduction>1</mechanicalReduction>
       </actuator>
@@ -118,8 +118,8 @@
       <type>transmission_interface/SimpleTransmission</type>
       <joint name="right_wheel_hinge">
-        <hardwareInterface>hardware_interface/EffortJointInterface</hardwareInterface>
+        <hardwareInterface>hardware_interface/VelocityJointInterface</hardwareInterface>
       </joint>
       <actuator name="motor2">
-        <hardwareInterface>hardware_interface/EffortJointInterface</hardwareInterface>
+        <hardwareInterface>hardware_interface/VelocityJointInterface</hardwareInterface>
         <mechanicalReduction>1</mechanicalReduction>
       </actuator>
