Commit message: solenoid plugin update

File: jetbot/jetbot_description/urdf/jetbot_rviz.xacro (robot description, xacro)
@@ -1,11 +1,4 @@
 <?xml version="1.0"?>
 <robot name="jetbot" xmlns:xacro="http://www.ros.org/wiki/xacro">
-    <xacro:include filename="$(find jetbot_description)/urdf/jetbot.gazebo" />
-    <!-- Used for fixing robot to Gazebo 'base_link' -->
-    <link name="world"/>
-    <joint name="fixed" type="fixed">
-      <parent link="world"/>
-      <child link="chassis"/>
-    </joint>
     <link name="chassis">
       <inertial>
@@ -111,23 +104,3 @@
     <link name="camera_link_optical">
     </link>
-    <transmission name="tran1">
-      <type>transmission_interface/SimpleTransmission</type>
-      <joint name="left_wheel_hinge">
-        <hardwareInterface>hardware_interface/VelocityJointInterface</hardwareInterface>
-      </joint>
-      <actuator name="motor1">
-        <hardwareInterface>hardware_interface/VelocityJointInterface</hardwareInterface>
-        <mechanicalReduction>1</mechanicalReduction>
-      </actuator>
-    </transmission>
-    <transmission name="tran2">
-      <type>transmission_interface/SimpleTransmission</type>
-      <joint name="right_wheel_hinge">
-        <hardwareInterface>hardware_interface/VelocityJointInterface</hardwareInterface>
-      </joint>
-      <actuator name="motor2">
-        <hardwareInterface>hardware_interface/VelocityJointInterface</hardwareInterface>
-        <mechanicalReduction>1</mechanicalReduction>
-      </actuator>
-    </transmission>
 </robot>

File: jetbot/jetbot_description/urdf/jetbot_soccer.xacro (robot description, xacro)
@@ -4238,5 +4238,5 @@
 		<child link="roller_stick_1" />
 		<axis xyz="-1 0 0"/>
-		<limit lower="-0.02" upper="0.05" effort="100" velocity="20" />
+		<limit lower="-0.01" upper="0.01" effort="30" velocity="200" />
 		<joint_properties friction="10.0"/>
 	</joint>

File: jetbot/jetbot_description/urdf/jetbot_soccer_rviz.xacro (robot description, xacro)
@@ -3,7 +3,8 @@
     <!-- Used for fixing jetbot_soccer to Gazebo 'base_link' -->
     <link name="world" />
-    <joint name="fixed" type="fixed">
+    <joint name="world_joint" type="fixed">
       <parent link="world"/>
       <child link="body_1"/>
+      <origin xyz="0.0 0.0 0.0" rpy="0.0 0.0 0.0" />
     </joint>
 	<link name="body_1">
@@ -1227,5 +1228,5 @@
 	</link>
 	<joint name="body_1_body_1_41_ova5647_housing_fixing" type="fixed">
-		<origin xyz="-0.280138 -0.345838 -0.0348527" rpy="-1.5708 1.34625 1.62107" />
+		<origin xyz="-0.280138 -0.345838 -0.0348527" rpy="-3.1416 2.91705 1.62107" />
 		<parent link="body_1" />
 		<child link="body_1_41_ova5647_housing" />
@@ -4243,5 +4244,5 @@
 		<child link="roller_stick_1" />
 		<axis xyz="-1 0 0"/>
-		<limit lower="-0.02" upper="0.02" effort="100" velocity="20" />
+		<limit lower="-0.01" upper="0.01" effort="100" velocity="20" />
 		<joint_properties friction="10.0"/>
 	</joint>
