Commit message: inertia update

File: jetbot/jetbot_description/urdf/jetbot_soccer_rviz.xacro (robot description, xacro)
@@ -10,24 +10,24 @@
 	<link name="body_1">
 		<inertial>
-			<origin xyz="0 0 0" rpy="0 0 0" />
-			<mass value="1e-9" />
-			<inertia ixx="0" ixy="0" ixz="0" iyy="0" iyz="0" izz="0" />
-		</inertial>
-	</link>
-	<link name="body_1_0_part_13">
-		<visual>
-			<geometry>
-				<mesh filename="file://$(find jetbot_description)/urdf/jetbot_soccer/part_13.stl"/>
-			</geometry>
-			<material name="body_1_0_part_13_material">
-				<color rgba="0.980392 0.713725 0.00392157 1.0"/>
-			</material>
-		</visual>
-		<collision>
-			<geometry>
-				<mesh filename="file://$(find jetbot_description)/urdf/jetbot_soccer/part_13.stl"/>
-			</geometry>
-			<material name="body_1_0_part_13_material">
-				<color rgba="0.980392 0.713725 0.00392157 1.0"/>
+			<origin xyz="0 0 0" rpy="0 0 0"/>
+			<mass value="1e-9" />
+			<inertia ixx="0" ixy="0" ixz="0" iyy="0" iyz="0" izz="0" />
+		</inertial>
+	</link>
+	<link name="body_1_12_part_1">
+		<visual>
+			<geometry>
+				<mesh filename="file://$(find jetbot_description)/urdf/jetbot_soccer/part_1.stl"/>
+			</geometry>
+			<material name="body_1_12_part_1_material">
+				<color rgba="0.25098 0.25098 0.25098 1.0"/>
+			</material>
+		</visual>
+		<collision>
+			<geometry>
+				<mesh filename="file://$(find jetbot_description)/urdf/jetbot_soccer/part_1.stl"/>
+			</geometry>
+			<material name="body_1_12_part_1_material">
+				<color rgba="0.25098 0.25098 0.25098 1.0"/>
 			</material>
 		</collision>
@@ -38,219 +38,74 @@
 		</inertial>
 	</link>
-	<joint name="body_1_body_1_0_part_13_fixing" type="fixed">
-		<origin xyz="-0.0599017 -0.223117 -0.0809911" rpy="3.14159 6.97139e-08 -1.54564" />
-		<parent link="body_1" />
-		<child link="body_1_0_part_13" />
-		<axis xyz="0 0 0"/>
-	</joint>
-	<link name="body_1_1_solenoid_body">
-		<visual>
-			<geometry>
-				<mesh filename="file://$(find jetbot_description)/urdf/jetbot_soccer/solenoid_body.stl"/>
-			</geometry>
-			<material name="body_1_1_solenoid_body_material">
-				<color rgba="0.647059 0.647059 0.647059 1.0"/>
-			</material>
-		</visual>
-		<collision>
-			<geometry>
-				<mesh filename="file://$(find jetbot_description)/urdf/jetbot_soccer/solenoid_body.stl"/>
-			</geometry>
-			<material name="body_1_1_solenoid_body_material">
-				<color rgba="0.647059 0.647059 0.647059 1.0"/>
-			</material>
-		</collision>
-		<inertial>
-			<origin xyz="0.0254 0.240515 0.144969" rpy="0 0 0"/>
-			<mass value="0.244615"/>
-			<inertia ixx="3.11153e-05" ixy="0"  ixz="0" iyy="6.81629e-05" iyz="0" izz="6.81629e-05" />
-		</inertial>
-	</link>
-	<joint name="body_1_body_1_1_solenoid_body_fixing" type="fixed">
-		<origin xyz="-0.522699 -0.257164 -0.281025" rpy="-5.12956e-06 7.06783e-08 -1.534" />
-		<parent link="body_1" />
-		<child link="body_1_1_solenoid_body" />
-		<axis xyz="0 0 0"/>
-	</joint>
-	<link name="body_1_2_motor">
-		<visual>
-			<geometry>
-				<mesh filename="file://$(find jetbot_description)/urdf/jetbot_soccer/motor.stl"/>
-			</geometry>
-			<material name="body_1_2_motor_material">
-				<color rgba="0.768627 0.886275 0.952941 1.0"/>
-			</material>
-		</visual>
-		<collision>
-			<geometry>
-				<mesh filename="file://$(find jetbot_description)/urdf/jetbot_soccer/motor.stl"/>
-			</geometry>
-			<material name="body_1_2_motor_material">
-				<color rgba="0.768627 0.886275 0.952941 1.0"/>
-			</material>
-		</collision>
-		<inertial>
-			<origin xyz="-4.35415e-05 -3.52147e-09 0.0124478" rpy="0 0 0"/>
-			<mass value="0.0092524"/>
-			<inertia ixx="7.38756e-07" ixy="-2.99969e-14"  ixz="-3.76571e-09" iyy="6.65816e-07" iyz="-4.40126e-13" izz="3.84144e-07" />
-		</inertial>
-	</link>
-	<joint name="body_1_body_1_2_motor_fixing" type="fixed">
-		<origin xyz="-0.318888 -0.263529 -0.10295" rpy="-1.5708 -8.32148e-08 -3.11644" />
-		<parent link="body_1" />
-		<child link="body_1_2_motor" />
-		<axis xyz="0 0 0"/>
-	</joint>
-	<link name="body_1_3_body_1">
-		<visual>
-			<geometry>
-				<mesh filename="file://$(find jetbot_description)/urdf/jetbot_soccer/body_1.stl"/>
-			</geometry>
-			<material name="body_1_3_body_1_material">
-				<color rgba="0.615686 0.811765 0.929412 1.0"/>
-			</material>
-		</visual>
-		<collision>
-			<geometry>
-				<mesh filename="file://$(find jetbot_description)/urdf/jetbot_soccer/body_1.stl"/>
-			</geometry>
-			<material name="body_1_3_body_1_material">
-				<color rgba="0.615686 0.811765 0.929412 1.0"/>
-			</material>
-		</collision>
-		<inertial>
-			<origin xyz="-0.0074183 0.00428296 0.00127" rpy="0 0 0"/>
-			<mass value="0.0641892"/>
-			<inertia ixx="0.000114848" ixy="-1.63955e-05"  ixz="0" iyy="9.59164e-05" iyz="0" izz="0.000210696" />
-		</inertial>
-	</link>
-	<joint name="body_1_body_1_3_body_1_fixing" type="fixed">
-		<origin xyz="-0.282828 -0.272179 -0.118531" rpy="3.14159 1.99925e-08 -2.05776" />
-		<parent link="body_1" />
-		<child link="body_1_3_body_1" />
-		<axis xyz="0 0 0"/>
-	</joint>
-	<link name="body_1_4_____.step">
-		<visual>
-			<geometry>
-				<mesh filename="file://$(find jetbot_description)/urdf/jetbot_soccer/____.step.stl"/>
-			</geometry>
-			<material name="body_1_4_____.step_material">
-				<color rgba="0.196078 0.207843 0.262745 1.0"/>
-			</material>
-		</visual>
-		<collision>
-			<geometry>
-				<mesh filename="file://$(find jetbot_description)/urdf/jetbot_soccer/____.step.stl"/>
-			</geometry>
-			<material name="body_1_4_____.step_material">
-				<color rgba="0.196078 0.207843 0.262745 1.0"/>
-			</material>
-		</collision>
-		<inertial>
-			<origin xyz="0.0566812 0.00635 0.0216284" rpy="0 0 0"/>
-			<mass value="1.66881e-05"/>
-			<inertia ixx="8.97864e-12" ixy="0"  ixz="9.36698e-14" iyy="4.1144e-11" iyz="0" izz="3.55308e-11" />
-		</inertial>
-	</link>
-	<joint name="body_1_body_1_4_____.step_fixing" type="fixed">
-		<origin xyz="-0.28264 -0.270685 -0.0526944" rpy="1.5708 -8.17417e-08 -3.09557" />
-		<parent link="body_1" />
-		<child link="body_1_4_____.step" />
-		<axis xyz="0 0 0"/>
-	</joint>
-	<link name="body_1_5_antenna_hub.step">
-		<visual>
-			<geometry>
-				<mesh filename="file://$(find jetbot_description)/urdf/jetbot_soccer/antenna_hub.step.stl"/>
-			</geometry>
-			<material name="body_1_5_antenna_hub.step_material">
-				<color rgba="0.666667 0.694118 0.764706 1.0"/>
-			</material>
-		</visual>
-		<collision>
-			<geometry>
-				<mesh filename="file://$(find jetbot_description)/urdf/jetbot_soccer/antenna_hub.step.stl"/>
-			</geometry>
-			<material name="body_1_5_antenna_hub.step_material">
-				<color rgba="0.666667 0.694118 0.764706 1.0"/>
-			</material>
-		</collision>
-		<inertial>
-			<origin xyz="0.057953 0.0136724 0.0389997" rpy="0 0 0"/>
-			<mass value="0.00502468"/>
-			<inertia ixx="3.59049e-07" ixy="1.69985e-09"  ixz="6.81694e-12" iyy="1.10073e-07" iyz="9.90347e-12" izz="3.57826e-07" />
-		</inertial>
-	</link>
-	<joint name="body_1_body_1_5_antenna_hub.step_fixing" type="fixed">
-		<origin xyz="-0.370701 -0.277526 -0.0486944" rpy="1.5708 -7.1782e-08 1.62107" />
-		<parent link="body_1" />
-		<child link="body_1_5_antenna_hub.step" />
-		<axis xyz="0 0 0"/>
-	</joint>
-	<link name="body_1_6_____.step">
-		<visual>
-			<geometry>
-				<mesh filename="file://$(find jetbot_description)/urdf/jetbot_soccer/____.step.stl"/>
-			</geometry>
-			<material name="body_1_6_____.step_material">
-				<color rgba="0.788235 0.788235 0.788235 1.0"/>
-			</material>
-		</visual>
-		<collision>
-			<geometry>
-				<mesh filename="file://$(find jetbot_description)/urdf/jetbot_soccer/____.step.stl"/>
-			</geometry>
-			<material name="body_1_6_____.step_material">
-				<color rgba="0.788235 0.788235 0.788235 1.0"/>
-			</material>
-		</collision>
-		<inertial>
-			<origin xyz="0.0566812 0.00635 0.0241684" rpy="0 0 0"/>
-			<mass value="1.66881e-05"/>
-			<inertia ixx="8.97864e-12" ixy="0"  ixz="9.36698e-14" iyy="4.1144e-11" iyz="0" izz="3.55308e-11" />
-		</inertial>
-	</link>
-	<joint name="body_1_body_1_6_____.step_fixing" type="fixed">
-		<origin xyz="-0.28264 -0.270685 -0.0526944" rpy="1.5708 -8.17417e-08 -3.09557" />
-		<parent link="body_1" />
-		<child link="body_1_6_____.step" />
-		<axis xyz="0 0 0"/>
-	</joint>
-	<link name="body_1_7_antenna_hub.step">
-		<visual>
-			<geometry>
-				<mesh filename="file://$(find jetbot_description)/urdf/jetbot_soccer/antenna_hub.step.stl"/>
-			</geometry>
-			<material name="body_1_7_antenna_hub.step_material">
-				<color rgba="0.666667 0.694118 0.764706 1.0"/>
-			</material>
-		</visual>
-		<collision>
-			<geometry>
-				<mesh filename="file://$(find jetbot_description)/urdf/jetbot_soccer/antenna_hub.step.stl"/>
-			</geometry>
-			<material name="body_1_7_antenna_hub.step_material">
-				<color rgba="0.666667 0.694118 0.764706 1.0"/>
-			</material>
-		</collision>
-		<inertial>
-			<origin xyz="0.057953 0.0136724 0.0389997" rpy="0 0 0"/>
-			<mass value="0.00502468"/>
-			<inertia ixx="3.59049e-07" ixy="1.69985e-09"  ixz="6.81694e-12" iyy="1.10073e-07" iyz="9.90347e-12" izz="3.57826e-07" />
-		</inertial>
-	</link>
-	<joint name="body_1_body_1_7_antenna_hub.step_fixing" type="fixed">
-		<origin xyz="-0.273229 -0.273176 -0.0486944" rpy="1.5708 -7.1782e-08 1.62107" />
-		<parent link="body_1" />
-		<child link="body_1_7_antenna_hub.step" />
-		<axis xyz="0 0 0"/>
-	</joint>
-	<link name="body_1_8_m3_l30mm">
+	<joint name="body_1_body_1_12_part_1_fixing" type="fixed">
+		<origin xyz="-0.280051 -0.342952 -0.0926791" rpy="6.97139e-08 8.32148e-08 0.0251544" />
+		<parent link="body_1" />
+		<child link="body_1_12_part_1" />
+		<axis xyz="0 0 0"/>
+	</joint>
+	<link name="body_1_13_m3_l35mm">
+		<visual>
+			<geometry>
+				<mesh filename="file://$(find jetbot_description)/urdf/jetbot_soccer/m3_l35mm.stl"/>
+			</geometry>
+			<material name="body_1_13_m3_l35mm_material">
+				<color rgba="0 0 0 1.0"/>
+			</material>
+		</visual>
+		<collision>
+			<geometry>
+				<mesh filename="file://$(find jetbot_description)/urdf/jetbot_soccer/m3_l35mm.stl"/>
+			</geometry>
+			<material name="body_1_13_m3_l35mm_material">
+				<color rgba="0 0 0 1.0"/>
+			</material>
+		</collision>
+		<inertial>
+			<origin xyz="0.17 -3.57955e-11 -0.0175" rpy="0 0 0"/>
+			<mass value="0.000921555"/>
+			<inertia ixx="8.78424e-08" ixy="5.12742e-15"  ixz="2.80925e-16" iyy="8.78424e-08" iyz="1.83386e-16" izz="3.55567e-09" />
+		</inertial>
+	</link>
+	<joint name="body_1_body_1_13_m3_l35mm_fixing" type="fixed">
+		<origin xyz="-0.0927726 -0.415205 -0.118531" rpy="3.14159 -1.06701e-07 2.65463" />
+		<parent link="body_1" />
+		<child link="body_1_13_m3_l35mm" />
+		<axis xyz="0 0 0"/>
+	</joint>
+	<link name="body_1_14_m3_l35mm">
+		<visual>
+			<geometry>
+				<mesh filename="file://$(find jetbot_description)/urdf/jetbot_soccer/m3_l35mm.stl"/>
+			</geometry>
+			<material name="body_1_14_m3_l35mm_material">
+				<color rgba="0 0 0 1.0"/>
+			</material>
+		</visual>
+		<collision>
+			<geometry>
+				<mesh filename="file://$(find jetbot_description)/urdf/jetbot_soccer/m3_l35mm.stl"/>
+			</geometry>
+			<material name="body_1_14_m3_l35mm_material">
+				<color rgba="0 0 0 1.0"/>
+			</material>
+		</collision>
+		<inertial>
+			<origin xyz="0.17 -3.57955e-11 -0.0175" rpy="0 0 0"/>
+			<mass value="0.000921555"/>
+			<inertia ixx="8.78424e-08" ixy="5.12742e-15"  ixz="2.80925e-16" iyy="8.78424e-08" iyz="1.83386e-16" izz="3.55567e-09" />
+		</inertial>
+	</link>
+	<joint name="body_1_body_1_14_m3_l35mm_fixing" type="fixed">
+		<origin xyz="-0.172405 -0.288254 -0.118531" rpy="3.14159 -1.06701e-07 2.65463" />
+		<parent link="body_1" />
+		<child link="body_1_14_m3_l35mm" />
+		<axis xyz="0 0 0"/>
+	</joint>
+	<link name="body_1_17_m3_l30mm">
 		<visual>
 			<geometry>
 				<mesh filename="file://$(find jetbot_description)/urdf/jetbot_soccer/m3_l30mm.stl"/>
 			</geometry>
-			<material name="body_1_8_m3_l30mm_material">
+			<material name="body_1_17_m3_l30mm_material">
 				<color rgba="0 0 0 1.0"/>
 			</material>
@@ -260,5 +115,5 @@
 				<mesh filename="file://$(find jetbot_description)/urdf/jetbot_soccer/m3_l30mm.stl"/>
 			</geometry>
-			<material name="body_1_8_m3_l30mm_material">
+			<material name="body_1_17_m3_l30mm_material">
 				<color rgba="0 0 0 1.0"/>
 			</material>
@@ -270,4 +125,236 @@
 		</inertial>
 	</link>
+	<joint name="body_1_body_1_17_m3_l30mm_fixing" type="fixed">
+		<origin xyz="-0.256915 -0.04564 -0.0812344" rpy="3.14159 7.1782e-08 -1.52052" />
+		<parent link="body_1" />
+		<child link="body_1_17_m3_l30mm" />
+		<axis xyz="0 0 0"/>
+	</joint>
+	<link name="body_1_18_m3_l30mm">
+		<visual>
+			<geometry>
+				<mesh filename="file://$(find jetbot_description)/urdf/jetbot_soccer/m3_l30mm.stl"/>
+			</geometry>
+			<material name="body_1_18_m3_l30mm_material">
+				<color rgba="0 0 0 1.0"/>
+			</material>
+		</visual>
+		<collision>
+			<geometry>
+				<mesh filename="file://$(find jetbot_description)/urdf/jetbot_soccer/m3_l30mm.stl"/>
+			</geometry>
+			<material name="body_1_18_m3_l30mm_material">
+				<color rgba="0 0 0 1.0"/>
+			</material>
+		</collision>
+		<inertial>
+			<origin xyz="0.16 -6.55175e-11 -0.015" rpy="0 0 0"/>
+			<mass value="0.000771083"/>
+			<inertia ixx="5.51132e-08" ixy="4.40552e-15"  ixz="2.36036e-16" iyy="5.51132e-08" iyz="1.55903e-16" izz="3.0332e-09" />
+		</inertial>
+	</link>
+	<joint name="body_1_body_1_18_m3_l30mm_fixing" type="fixed">
+		<origin xyz="-0.33177 -0.0489804 -0.0812344" rpy="3.14159 7.1782e-08 -1.52052" />
+		<parent link="body_1" />
+		<child link="body_1_18_m3_l30mm" />
+		<axis xyz="0 0 0"/>
+	</joint>
+	<link name="body_1_23_m3_l35mm">
+		<visual>
+			<geometry>
+				<mesh filename="file://$(find jetbot_description)/urdf/jetbot_soccer/m3_l35mm.stl"/>
+			</geometry>
+			<material name="body_1_23_m3_l35mm_material">
+				<color rgba="0 0 0 1.0"/>
+			</material>
+		</visual>
+		<collision>
+			<geometry>
+				<mesh filename="file://$(find jetbot_description)/urdf/jetbot_soccer/m3_l35mm.stl"/>
+			</geometry>
+			<material name="body_1_23_m3_l35mm_material">
+				<color rgba="0 0 0 1.0"/>
+			</material>
+		</collision>
+		<inertial>
+			<origin xyz="0.17 -3.57955e-11 -0.0175" rpy="0 0 0"/>
+			<mass value="0.000921555"/>
+			<inertia ixx="8.78424e-08" ixy="5.12742e-15"  ixz="2.80925e-16" iyy="8.78424e-08" iyz="1.83386e-16" izz="3.55567e-09" />
+		</inertial>
+	</link>
+	<joint name="body_1_body_1_23_m3_l35mm_fixing" type="fixed">
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
File: jetbot/jetbot_description/urdf/jetbot_soccer_test.xacro (robot description, xacro)
@@ -1,5 +1,5 @@
 <?xml version="1.0"?>
 <robot name="jetbot_soccer" xmlns:xacro="http://www.ros.org/wiki/xacro">
-	<xacro:include filename="$(find jetbot_description)/urdf/jetbot_soccer.gazebo" />
+	<xacro:include filename="$(find jetbot_description)/urdf/jetbot_soccer_test.gazebo" />
 	<link name="body_1">
 		<inertial>
@@ -543,5 +543,5 @@
 		<child link="roller_stick_1" />
 		<axis xyz="-1 0 0"/>
-		<limit lower="0.01" upper="0.04" effort="30" velocity="200" />
+		<limit lower="-0.01" upper="0.01" effort="30" velocity="200" />
 		<joint_properties friction="10.0"/>
 	</joint>
@@ -4223,23 +4223,3 @@
       </actuator>
     </transmission>
-    <transmission name="tran5">
-      <type>transmission_interface/SimpleTransmission</type>
-      <joint name="roller">
-        <hardwareInterface>hardware_interface/VelocityJointInterface</hardwareInterface>
-      </joint>
-      <actuator name="motor5">
-        <hardwareInterface>hardware_interface/VelocityJointInterface</hardwareInterface>
-        <mechanicalReduction>1</mechanicalReduction>
-      </actuator>
-    </transmission>
-    <transmission name="tran6">
-	  <type>transmission_interface/SimpleTransmission</type>
-	  <joint name="stick">
-	    <hardwareInterface>hardware_interface/VelocityJointInterface</hardwareInterface>
-	  </joint>
-	  <actuator name="lift_motor">
-	    <hardwareInterface>hardware_interface/VelocityJointInterface</hardwareInterface>
-	    <mechanicalReduction>1</mechanicalReduction>
-	  </actuator>
-  	</transmission>
 </robot>
