Commit message: Control by ROS topic update

File: jetbot/jetbot_description/urdf/jetbot_soccer.xacro (robot description, xacro)
@@ -1,4 +1,5 @@
 <?xml version="1.0"?>
-<robot name="onshape" xmlns:xacro="http://www.ros.org/wiki/xacro">
+<robot name="jetbot_soccer" xmlns:xacro="http://www.ros.org/wiki/xacro">
+	<xacro:include filename="$(find jetbot_description)/urdf/jetbot_soccer.gazebo" />
 	<link name="body_1">
 		<inertial>
@@ -84,7 +85,7 @@
 		</collision>
 		<inertial>
-			<origin xyz="4.83699e-18 -2.58534e-16 0.0170962" rpy="0 0 0"/>
-			<mass value="0.0218513"/>
-			<inertia ixx="3.91997e-06" ixy="0"  ixz="0" iyy="3.66242e-06" iyz="0" izz="1.61449e-06" />
+			<origin xyz="0 0 0" rpy="0 0 0"/>
+			<mass value="0"/>
+			<inertia ixx="0" ixy="0"  ixz="0" iyy="0" iyz="0" izz="0" />
 		</inertial>
 	</link>
@@ -95,10 +96,10 @@
 		<axis xyz="0 0 0"/>
 	</joint>
-	<link name="body_1_3_m3_l30mm">
-		<visual>
-			<geometry>
-				<mesh filename="file://$(find jetbot_description)/urdf/jetbot_soccer/m3_l30mm.stl"/>
-			</geometry>
-			<material name="body_1_3_m3_l30mm_material">
+	<link name="body_1_3_document">
+		<visual>
+			<geometry>
+				<mesh filename="file://$(find jetbot_description)/urdf/jetbot_soccer/document.stl"/>
+			</geometry>
+			<material name="body_1_3_document_material">
 				<color rgba="0 0 0 1.0"/>
 			</material>
@@ -106,20 +107,20 @@
 		<collision>
 			<geometry>
-				<mesh filename="file://$(find jetbot_description)/urdf/jetbot_soccer/m3_l30mm.stl"/>
-			</geometry>
-			<material name="body_1_3_m3_l30mm_material">
+				<mesh filename="file://$(find jetbot_description)/urdf/jetbot_soccer/document.stl"/>
+			</geometry>
+			<material name="body_1_3_document_material">
 				<color rgba="0 0 0 1.0"/>
 			</material>
 		</collision>
 		<inertial>
-			<origin xyz="0.16 -6.55175e-11 -0.015" rpy="0 0 0"/>
-			<mass value="0.000771083"/>
-			<inertia ixx="5.51132e-08" ixy="4.40552e-15"  ixz="2.36036e-16" iyy="5.51132e-08" iyz="1.55903e-16" izz="3.0332e-09" />
-		</inertial>
-	</link>
-	<joint name="body_1_body_1_3_m3_l30mm_fixing" type="fixed">
+			<origin xyz="0 0 0" rpy="0 0 0"/>
+			<mass value="0"/>
+			<inertia ixx="0" ixy="0"  ixz="0" iyy="0" iyz="0" izz="0" />
+		</inertial>
+	</link>
+	<joint name="body_1_body_1_3_document_fixing" type="fixed">
 		<origin xyz="-0.141841 -0.014347 -0.0297213" rpy="-3.14159 1.35133e-16 -0.523599" />
 		<parent link="body_1" />
-		<child link="body_1_3_m3_l30mm" />
+		<child link="body_1_3_document" />
 		<axis xyz="0 0 0"/>
 	</joint>
@@ -142,7 +143,7 @@
 		</collision>
 		<inertial>
-			<origin xyz="0.18 -1.5606e-11 -0.02" rpy="0 0 0"/>
-			<mass value="0.00107203"/>
-			<inertia ixx="1.32091e-07" ixy="5.85025e-15"  ixz="3.17107e-16" iyy="1.32091e-07" iyz="2.04825e-16" izz="4.07814e-09" />
+			<origin xyz="0 0 0" rpy="0 0 0"/>
+			<mass value="0"/>
+			<inertia ixx="0" ixy="0"  ixz="0" iyy="0" iyz="0" izz="0" />
 		</inertial>
 	</link>
@@ -171,7 +172,7 @@
 		</collision>
 		<inertial>
-			<origin xyz="0.0566812 0.00635 0.0216284" rpy="0 0 0"/>
-			<mass value="1.66881e-05"/>
-			<inertia ixx="8.97864e-12" ixy="0"  ixz="9.36698e-14" iyy="4.1144e-11" iyz="0" izz="3.55308e-11" />
+			<origin xyz="0 0 0" rpy="0 0 0"/>
+			<mass value="0"/>
+			<inertia ixx="0" ixy="0"  ixz="0" iyy="0" iyz="0" izz="0" />
 		</inertial>
 	</link>
@@ -200,7 +201,7 @@
 		</collision>
 		<inertial>
-			<origin xyz="0.057953 0.0136724 0.0389997" rpy="0 0 0"/>
-			<mass value="0.00502468"/>
-			<inertia ixx="3.59049e-07" ixy="1.69985e-09"  ixz="6.81694e-12" iyy="1.10073e-07" iyz="9.90347e-12" izz="3.57826e-07" />
+			<origin xyz="0 0 0" rpy="0 0 0"/>
+			<mass value="0"/>
+			<inertia ixx="0" ixy="0"  ixz="0" iyy="0" iyz="0" izz="0" />
 		</inertial>
 	</link>
@@ -229,7 +230,7 @@
 		</collision>
 		<inertial>
-			<origin xyz="0.0566812 0.00635 0.0241684" rpy="0 0 0"/>
-			<mass value="1.66881e-05"/>
-			<inertia ixx="8.97864e-12" ixy="0"  ixz="9.36698e-14" iyy="4.1144e-11" iyz="0" izz="3.55308e-11" />
+			<origin xyz="0 0 0" rpy="0 0 0"/>
+			<mass value="0"/>
+			<inertia ixx="0" ixy="0"  ixz="0" iyy="0" iyz="0" izz="0" />
 		</inertial>
 	</link>
@@ -258,7 +259,7 @@
 		</collision>
 		<inertial>
-			<origin xyz="0.057953 0.0136724 0.0389997" rpy="0 0 0"/>
-			<mass value="0.00502468"/>
-			<inertia ixx="3.59049e-07" ixy="1.69985e-09"  ixz="6.81694e-12" iyy="1.10073e-07" iyz="9.90347e-12" izz="3.57826e-07" />
+			<origin xyz="0 0 0" rpy="0 0 0"/>
+			<mass value="0"/>
+			<inertia ixx="0" ixy="0"  ixz="0" iyy="0" iyz="0" izz="0" />
 		</inertial>
 	</link>
@@ -316,7 +317,7 @@
 		</collision>
 		<inertial>
-			<origin xyz="0.0566812 0.00635 0.0190884" rpy="0 0 0"/>
-			<mass value="1.66881e-05"/>
-			<inertia ixx="8.97864e-12" ixy="0"  ixz="9.36698e-14" iyy="4.1144e-11" iyz="0" izz="3.55308e-11" />
+			<origin xyz="0 0 0" rpy="0 0 0"/>
+			<mass value="0"/>
+			<inertia ixx="0" ixy="0"  ixz="0" iyy="0" iyz="0" izz="0" />
 		</inertial>
 	</link>
@@ -345,7 +346,7 @@
 		</collision>
 		<inertial>
-			<origin xyz="0.18 -1.5606e-11 -0.02" rpy="0 0 0"/>
-			<mass value="0.00107203"/>
-			<inertia ixx="1.32091e-07" ixy="5.85025e-15"  ixz="3.17107e-16" iyy="1.32091e-07" iyz="2.04825e-16" izz="4.07814e-09" />
+			<origin xyz="0 0 0" rpy="0 0 0"/>
+			<mass value="0"/>
+			<inertia ixx="0" ixy="0"  ixz="0" iyy="0" iyz="0" izz="0" />
 		</inertial>
 	</link>
@@ -385,10 +386,10 @@
 		<axis xyz="0 0 0"/>
 	</joint>
-	<link name="body_1_13_m3_l30mm">
-		<visual>
-			<geometry>
-				<mesh filename="file://$(find jetbot_description)/urdf/jetbot_soccer/m3_l30mm.stl"/>
-			</geometry>
-			<material name="body_1_13_m3_l30mm_material">
+	<link name="body_1_13_document">
+		<visual>
+			<geometry>
+				<mesh filename="file://$(find jetbot_description)/urdf/jetbot_soccer/document.stl"/>
+			</geometry>
+			<material name="body_1_13_document_material">
 				<color rgba="0 0 0 1.0"/>
 			</material>
@@ -396,20 +397,20 @@
 		<collision>
 			<geometry>
-				<mesh filename="file://$(find jetbot_description)/urdf/jetbot_soccer/m3_l30mm.stl"/>
-			</geometry>
-			<material name="body_1_13_m3_l30mm_material">
+				<mesh filename="file://$(find jetbot_description)/urdf/jetbot_soccer/document.stl"/>
+			</geometry>
+			<material name="body_1_13_document_material">
 				<color rgba="0 0 0 1.0"/>
 			</material>
 		</collision>
 		<inertial>
-			<origin xyz="0.16 -6.55175e-11 -0.015" rpy="0 0 0"/>
-			<mass value="0.000771083"/>
-			<inertia ixx="5.51132e-08" ixy="4.40552e-15"  ixz="2.36036e-16" iyy="5.51132e-08" iyz="1.55903e-16" izz="3.0332e-09" />
-		</inertial>
-	</link>
-	<joint name="body_1_body_1_13_m3_l30mm_fixing" type="fixed">
+			<origin xyz="0 0 0" rpy="0 0 0"/>
+			<mass value="0"/>
+			<inertia ixx="0" ixy="0"  ixz="0" iyy="0" iyz="0" izz="0" />
+		</inertial>
+	</link>
+	<joint name="body_1_body_1_13_document_fixing" type="fixed">
 		<origin xyz="-0.143222 0.115428 -0.0297213" rpy="-3.14159 1.35133e-16 -0.523599" />
 		<parent link="body_1" />
-		<child link="body_1_13_m3_l30mm" />
+		<child link="body_1_13_document" />
 		<axis xyz="0 0 0"/>
 	</joint>
@@ -432,7 +433,7 @@
 		</collision>
 		<inertial>
-			<origin xyz="0.0431301 0.0303966 0.0091596" rpy="0 0 0"/>
-			<mass value="0.313249"/>
-			<inertia ixx="0.000145269" ixy="-1.186e-05"  ixz="1.72812e-06" iyy="0.000198778" iyz="-2.02085e-05" izz="0.000304634" />
+			<origin xyz="0 0 0" rpy="0 0 0"/>
+			<mass value="0"/>
+			<inertia ixx="0" ixy="0"  ixz="0" iyy="0" iyz="0" izz="0" />
 		</inertial>
 	</link>
@@ -461,7 +462,7 @@
 		</collision>
 		<inertial>
-			<origin xyz="-0.0228199 -0.236326 -0.0239225" rpy="0 0 0"/>
-			<mass value="0.096502"/>
-			<inertia ixx="0.000181039" ixy="-2.80846e-05"  ixz="-1.52129e-07" iyy="0.000148471" iyz="8.69589e-08" izz="0.000327931" />
+			<origin xyz="0 0 0" rpy="0 0 0"/>
+			<mass value="0"/>
+			<inertia ixx="0" ixy="0"  ixz="0" iyy="0" iyz="0" izz="0" />
 		</inertial>
 	</link>
@@ -472,10 +473,10 @@
 		<axis xyz="0 0 0"/>
 	</joint>
-	<link name="body_1_16_m3_l30mm">
-		<visual>
-			<geometry>
-				<mesh filename="file://$(find jetbot_description)/urdf/jetbot_soccer/m3_l30mm.stl"/>
-			</geometry>
-			<material name="body_1_16_m3_l30mm_material">
+	<link name="body_1_16_document">
+		<visual>
+			<geometry>
+				<mesh filename="file://$(find jetbot_description)/urdf/jetbot_soccer/document.stl"/>
+			</geometry>
+			<material name="body_1_16_document_material">
 				<color rgba="0 0 0 1.0"/>
 			</material>
@@ -483,20 +484,20 @@
 		<collision>
 			<geometry>
-				<mesh filename="file://$(find jetbot_description)/urdf/jetbot_soccer/m3_l30mm.stl"/>
-			</geometry>
-			<material name="body_1_16_m3_l30mm_material">
+				<mesh filename="file://$(find jetbot_description)/urdf/jetbot_soccer/document.stl"/>
+			</geometry>
+			<material name="body_1_16_document_material">
 				<color rgba="0 0 0 1.0"/>
 			</material>
 		</collision>
 		<inertial>
-			<origin xyz="0.16 -6.55175e-11 -0.015" rpy="0 0 0"/>
-			<mass value="0.000771083"/>
-			<inertia ixx="5.51132e-08" ixy="4.40552e-15"  ixz="2.36036e-16" iyy="5.51132e-08" iyz="1.55903e-16" izz="3.0332e-09" />
-		</inertial>
-	</link>
-	<joint name="body_1_body_1_16_m3_l30mm_fixing" type="fixed">
+			<origin xyz="0 0 0" rpy="0 0 0"/>
+			<mass value="0"/>
+			<inertia ixx="0" ixy="0"  ixz="0" iyy="0" iyz="0" izz="0" />
+		</inertial>
+	</link>
+	<joint name="body_1_body_1_16_document_fixing" type="fixed">
 		<origin xyz="-0.0682963 0.116225 -0.0297213" rpy="-3.14159 1.35133e-16 -0.523599" />
 		<parent link="body_1" />
-		<child link="body_1_16_m3_l30mm" />
+		<child link="body_1_16_document" />
 		<axis xyz="0 0 0"/>
 	</joint>
@@ -519,7 +520,7 @@
 		</collision>
 		<inertial>
-			<origin xyz="0.0579666 0.0092 0.021663" rpy="0 0 0"/>
-			<mass value="1.44368e-05"/>
-			<inertia ixx="1.51981e-10" ixy="0"  ixz="-1.79403e-15" iyy="2.13123e-12" iyz="0" izz="1.51976e-10" />
+			<origin xyz="0 0 0" rpy="0 0 0"/>
+			<mass value="0"/>
+			<inertia ixx="0" ixy="0"  ixz="0" iyy="0" iyz="0" izz="0" />
 		</inertial>
 	</link>
@@ -548,7 +549,7 @@
 		</collision>
 		<inertial>
-			<origin xyz="0.00115354 0.0049 -0.000292476" rpy="0 0 0"/>
-			<mass value="0.022861"/>
-			<inertia ixx="1.1405e-05" ixy="2.57626e-16"  ixz="6.63789e-09" iyy="3.74833e-05" iyz="4.54387e-16" izz="2.60906e-05" />
+			<origin xyz="0 0 0" rpy="0 0 0"/>
+			<mass value="0"/>
+			<inertia ixx="0" ixy="0"  ixz="0" iyy="0" iyz="0" izz="0" />
 		</inertial>
 	</link>
@@ -577,7 +578,7 @@
 		</collision>
 		<inertial>
-			<origin xyz="0.0554267 0.0092 0.021663" rpy="0 0 0"/>
-			<mass value="1.44368e-05"/>
-			<inertia ixx="1.51981e-10" ixy="0"  ixz="-1.79403e-15" iyy="2.13123e-12" iyz="0" izz="1.51976e-10" />
+			<origin xyz="0 0 0" rpy="0 0 0"/>
+			<mass value="0"/>
+			<inertia ixx="0" ixy="0"  ixz="0" iyy="0" iyz="0" izz="0" />
 		</inertial>
 	</link>
@@ -606,7 +607,7 @@
 		</collision>
 		<inertial>
-			<origin xyz="0.0579666 0.0092 0.019123" rpy="0 0 0"/>
-			<mass value="1.44368e-05"/>
-			<inertia ixx="1.51981e-10" ixy="0"  ixz="-1.79403e-15" iyy="2.13123e-12" iyz="0" izz="1.51976e-10" />
+			<origin xyz="0 0 0" rpy="0 0 0"/>
+			<mass value="0"/>
+			<inertia ixx="0" ixy="0"  ixz="0" iyy="0" iyz="0" izz="0" />
 		</inertial>
 	</link>
@@ -635,7 +636,7 @@
 		</collision>
 		<inertial>
-			<origin xyz="-0.0170541 -0.296506 -0.00120586" rpy="0 0 0"/>
-			<mass value="0.0568507"/>
-			<inertia ixx="8.73711e-06" ixy="-2.19732e-07"  ixz="1.45771e-08" iyy="1.38518e-05" iyz="1.91693e-09" izz="1.6021e-05" />
+			<origin xyz="0 0 0" rpy="0 0 0"/>
+			<mass value="0"/>
+			<inertia ixx="0" ixy="0"  ixz="0" iyy="0" iyz="0" izz="0" />
 		</inertial>
 	</link>
@@ -664,7 +665,7 @@
 		</collision>
 		<inertial>
-			<origin xyz="0.00281781 -0.001 -0.00411411" rpy="0 0 0"/>
-			<mass value="0.000473713"/>
-			<inertia ixx="4.49035e-09" ixy="0"  ixz="0" iyy="3.87759e-09" iyz="0" izz="7.28246e-09" />
+			<origin xyz="0 0 0" rpy="0 0 0"/>
+			<mass value="0"/>
+			<inertia ixx="0" ixy="0"  ixz="0" iyy="0" iyz="0" izz="0" />
 		</inertial>
 	</link>
@@ -693,7 +694,7 @@
 		</collision>
 		<inertial>
-			<origin xyz="0.0578996 0.0921429 0.0389994" rpy="0 0 0"/>
-			<mass value="0.0180219"/>
-			<inertia ixx="3.50659e-05" ixy="-1.16532e-07"  ixz="4.17062e-11" iyy="2.77141e-07" iyz="-6.64058e-10" izz="3.50587e-05" />
+			<origin xyz="0 0 0" rpy="0 0 0"/>
+			<mass value="0"/>
+			<inertia ixx="0" ixy="0"  ixz="0" iyy="0" iyz="0" izz="0" />
 		</inertial>
 	</link>
@@ -722,7 +723,7 @@
 		</collision>
 		<inertial>
-			<origin xyz="0.0578996 0.0921429 0.0389994" rpy="0 0 0"/>
-			<mass value="0.0180219"/>
-			<inertia ixx="3.50659e-05" ixy="-1.16532e-07"  ixz="4.17062e-11" iyy="2.77141e-07" iyz="-6.64058e-10" izz="3.50587e-05" />
+			<origin xyz="0 0 0" rpy="0 0 0"/>
+			<mass value="0"/>
+			<inertia ixx="0" ixy="0"  ixz="0" iyy="0" iyz="0" izz="0" />
 		</inertial>
 	</link>
@@ -751,7 +752,7 @@
 		</collision>
 		<inertial>
-			<origin xyz="-0.000399961 0.0109757 -0.000299917" rpy="0 0 0"/>
-			<mass value="0.0249892"/>
-			<inertia ixx="1.87787e-05" ixy="-9.12923e-12"  ixz="3.19582e-12" iyy="2.66904e-05" iyz="-2.04002e-11" izz="9.41616e-06" />
+			<origin xyz="0 0 0" rpy="0 0 0"/>
+			<mass value="0"/>
+			<inertia ixx="0" ixy="0"  ixz="0" iyy="0" iyz="0" izz="0" />
 		</inertial>
 	</link>
@@ -780,7 +781,7 @@
 		</collision>
 		<inertial>
-			<origin xyz="0.0554267 0.0092 0.019123" rpy="0 0 0"/>
-			<mass value="1.44368e-05"/>
-			<inertia ixx="1.51981e-10" ixy="0"  ixz="-1.79403e-15" iyy="2.13123e-12" iyz="0" izz="1.51976e-10" />
+			<origin xyz="0 0 0" rpy="0 0 0"/>
+			<mass value="0"/>
+			<inertia ixx="0" ixy="0"  ixz="0" iyy="0" iyz="0" izz="0" />
 		</inertial>
 	</link>
@@ -809,7 +810,7 @@
 		</collision>
 		<inertial>
-			<origin xyz="-0.0747424 -0.260504 -0.00127328" rpy="0 0 0"/>
-			<mass value="0.0568507"/>
-			<inertia ixx="1.27634e-05" ixy="2.10488e-06"  ixz="5.62847e-09" iyy="9.8255e-06" iyz="-1.35826e-08" izz="1.6021e-05" />
+			<origin xyz="0 0 0" rpy="0 0 0"/>
+			<mass value="0"/>
+			<inertia ixx="0" ixy="0"  ixz="0" iyy="0" iyz="0" izz="0" />
 		</inertial>
 	</link>
@@ -820,10 +821,10 @@
 		<axis xyz="0 0 0"/>
 	</joint>
-	<link name="body_1_28_m3_l30mm">
-		<visual>
-			<geometry>
-				<mesh filename="file://$(find jetbot_description)/urdf/jetbot_soccer/m3_l30mm.stl"/>
-			</geometry>
-			<material name="body_1_28_m3_l30mm_material">
+	<link name="body_1_28_document">
+		<visual>
+			<geometry>
+				<mesh filename="file://$(find jetbot_description)/urdf/jetbot_soccer/document.stl"/>
+			</geometry>
+			<material name="body_1_28_document_material">
 				<color rgba="0 0 0 1.0"/>
 			</material>
@@ -831,20 +832,20 @@
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
File: jetbot/jetbot_description/urdf/jetbot_soccer_rviz.xacro (robot description, xacro)
@@ -8,9 +8,9 @@
     </joint>
 	<link name="body_1">
-	<inertial>
-		<origin xyz="0 0 0" rpy="0 0 0" />
-		<mass value="1e-9" />
-		<inertia ixx="0" ixy="0" ixz="0" iyy="0" iyz="0" izz="0" />
-	</inertial>
+		<inertial>
+			<origin xyz="0 0 0" rpy="0 0 0" />
+			<mass value="1e-9" />
+			<inertia ixx="0" ixy="0" ixz="0" iyy="0" iyz="0" izz="0" />
+		</inertial>
 	</link>
 	<link name="body_1_0_body_3">

Commit message: omniwheel subwheel update new

File: jetbot/jetbot_description/urdf/jetbot_soccer.xacro (robot description, xacro)
@@ -4180,6 +4180,6 @@
 		<child link="roller_stick_1" />
 		<axis xyz="-1 0 0"/>
-		<limit lower="-1e+16" upper="1e+16" effort="1.5" velocity="50" />
-		<joint_properties friction="0.0"/>
+		<limit lower="-0.02" upper="0.08" effort="50" velocity="100" />
+		<joint_properties friction="100.0"/>
 	</joint>
 	<transmission name="tran1">

Commit message: Add files via upload
Steering unbalance problem solve

File: jetbot/jetbot_description/urdf/jetbot_soccer.xacro (robot description, xacro)
@@ -4224,5 +4224,5 @@
 			<origin xyz="0.04445 0.29536 0.137105" rpy="0 0 0"/>
 			<mass value="0.0115774"/>
-			<inertia ixx="1.72634e-07" ixy="0"  ixz="0" iyy="7.7112e-06" iyz="0" izz="7.7112e-06" />
+			<inertia ixx="0" ixy="0"  ixz="0" iyy="0" iyz="0" izz="0" />
 		</inertial>
 	</link>
@@ -4244,8 +4244,8 @@
       <type>transmission_interface/SimpleTransmission</type>
       <joint name="wheel1">
-        <hardwareInterface>hardware_interface/VelocityJointInterface</hardwareInterface>
+        <hardwareInterface>EffortJointInterface</hardwareInterface>
       </joint>
       <actuator name="motor1">
-        <hardwareInterface>hardware_interface/VelocityJointInterface</hardwareInterface>
+        <hardwareInterface>EffortJointInterface</hardwareInterface>
         <mechanicalReduction>1</mechanicalReduction>
       </actuator>
@@ -4254,8 +4254,8 @@
       <type>transmission_interface/SimpleTransmission</type>
       <joint name="wheel2">
-        <hardwareInterface>hardware_interface/VelocityJointInterface</hardwareInterface>
+        <hardwareInterface>EffortJointInterface</hardwareInterface>
       </joint>
       <actuator name="motor2">
-        <hardwareInterface>hardware_interface/VelocityJointInterface</hardwareInterface>
+        <hardwareInterface>EffortJointInterface</hardwareInterface>
         <mechanicalReduction>1</mechanicalReduction>
       </actuator>
@@ -4264,8 +4264,8 @@
       <type>transmission_interface/SimpleTransmission</type>
       <joint name="wheel3">
-        <hardwareInterface>hardware_interface/VelocityJointInterface</hardwareInterface>
+        <hardwareInterface>EffortJointInterface</hardwareInterface>
       </joint>
       <actuator name="motor3">
-        <hardwareInterface>hardware_interface/VelocityJointInterface</hardwareInterface>
+        <hardwareInterface>EffortJointInterface</hardwareInterface>
         <mechanicalReduction>1</mechanicalReduction>
       </actuator>
@@ -4274,8 +4274,8 @@
       <type>transmission_interface/SimpleTransmission</type>
       <joint name="wheel4">
-        <hardwareInterface>hardware_interface/VelocityJointInterface</hardwareInterface>
+        <hardwareInterface>EffortJointInterface</hardwareInterface>
       </joint>
       <actuator name="motor4">
-        <hardwareInterface>hardware_interface/VelocityJointInterface</hardwareInterface>
+        <hardwareInterface>EffortJointInterface</hardwareInterface>
         <mechanicalReduction>1</mechanicalReduction>
       </actuator>

Commit message: solenoid kicker update

File: jetbot/jetbot_description/urdf/jetbot_soccer.xacro (robot description, xacro)
@@ -543,6 +543,6 @@
 		<child link="roller_stick_1" />
 		<axis xyz="-1 0 0"/>
-		<limit lower="0.01" upper="0.04" effort="30" velocity="200" />
-		<joint_properties friction="10.0"/>
+		<limit lower="-0.02" upper="0.04" effort="30" velocity="30" />
+		<joint_properties friction="1.0"/>
 	</joint>
 	<link name="body_1_22_pcb.step">

Commit message: ForgER update

File: jetbot/jetbot_description/urdf/jetbot_soccer.xacro (robot description, xacro)
@@ -2511,4 +2511,29 @@
 		<joint_properties friction="0.0"/>
 	</joint>
+	<xacro:property name="camera_link" value="0.001" /> <!-- Size of square 'camera' box -->
+	<joint name="camera_joint" type="fixed">
+    	<axis xyz="0 0 1"/>
+    	<origin xyz="0.00202223 -0.0745669 -0.0321728" rpy="0 0.3 -1.52052" />
+    	<parent link="rspcameramia_1"/>
+    	<child link="camera_link"/>
+  	</joint>
+	<!-- IR -->
+	<link name="camera_link">
+		<collision>
+	    	<origin xyz="0 0 0" rpy="0 0 0"/>
+	    	<geometry>
+	    		<box size="${camera_link} ${camera_link} ${camera_link}"/>
+	      	</geometry>
+	    </collision>
+	    <visual>
+	    	<origin xyz="0 0 0" rpy="0 0 0"/>
+	     	<material name="red"/>
+	    </visual>
+	    <inertial>
+	    	<mass value="1e-5" />
+	     	<origin xyz="0 0 0" rpy="0 0 0"/>
+	     	<inertia ixx="1e-6" ixy="0" ixz="0" iyy="1e-6" iyz="0" izz="1e-6" />
+	  	</inertial>
+	</link>
 	<link name="ir_sensor_1">
 		<collision>
