Commit message: Add files via upload
Roller speed limit, friction parameter update

File: deepsoccer_pc/deepsoccer_description/urdf/deepsoccer_1.xacro (robot description, xacro)
@@ -318,5 +318,5 @@
 		<child link="roller_1" />
 		<axis xyz="-1 0 0"/>
-		<limit lower="-1e+16" upper="1e+16" effort="1.5" velocity="200" />
+		<limit lower="-1e+16" upper="1e+16" effort="1.5" velocity="1000" />
 		<joint_properties friction="0.0"/>
 	</joint>
